File: projects/nrf24l01breakout/nrf24l01brekaout/nrf2401breakout.sch (KiCad schematic (older format))
At the start: 8 parts, among them J1 Conn_01x02, U1 LM1117-3.3

Commit message: upd PCB thene
Parts:
- added J2, J3: Conn_01x04_Male, Pin_Headers:Pin_Header_Straight_1x04_Pitch2.54mm, symbol Connector:Conn_01x04_Male
- added U2: nRF24L01, symbol miscomponentes:nRF24L01
- C1: footprint (none) -> Capacitors_SMD:CP_Elec_4x5.7
- C2, C4: footprint (none) -> Capacitors_SMD:C_0603_HandSoldering
- C3: footprint (none) -> Capacitors_SMD:C_0805_HandSoldering
- D1: footprint (none) -> Diodes_SMD:D_0603
- J1: footprint (none) -> Connectors_JST:JST_EH_S02B-EH_02x2.50mm_Angled
- R1: footprint (none) -> Resistors_SMD:R_0603_HandSoldering
Connections:
- net labels added: CE, IRQ, MISO, MOSI, SCK, ~CSN
- wire segments 31 -> 48
Other:
- note added: "Conectores"
- note added: "Fuente de potencia"
- note added: "Módulo nRF24l01"
- note added: "The nRF24L01+ are RF transceiver modules that can be used\nfor wireless communications. They operate at a voltage \nrange of 1.9 – 3.6V for power. This nRF24L01 breakout \nadapter can be powered off 5V-12V and supplies well \nregulated 3.3V to the NRF24L01 socket. It also breaks \nout the pins for easier hookup and has a power on LED."
- note added: "nRF24l01"
- moved on the sheet: U1
